File: MiniShieldMWC.sch (EAGLE design)
At the start: 24 parts

Commit message: 1.1
Connections:
- net P$1 renamed N$19
Changed lines of the file:
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@@
 </segment>
 </net>
-<net name="P$1" class="0">
+<net name="N$19" class="0">
 <segment>
 <pinref part="U$3" gate="G$1" pin="VIN"/>
